File: mini-truss-pcb/truss_PCB/bridge_driver0_sch.kicad_sch (KiCad schematic)
At the start: 16 parts, among them J7 IN_B, Q3 BC807, U3 HX711

Commit message: added basic firmware tests
Parts:
- renumbered C7 to C1, C8 to C2, C9 to C3, EC5 to EC1, EC6 to EC2, J7 to J5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
